File: PCB + Schematic/gpsBreakout/_autosave-gpsBreakout.kicad_pcb (KiCad board)
At the start: 2 copper layers, 24.8 x 26.5 mm, 17 parts, among them J1 Header, U1 ATGM336H, U2 AT24CS32-STUM, U3 AT2659

Commit message: Routing!
Parts:
- moved C3 0.63 mm to (150.7, 87.9)
- moved U3 0.63 mm to (152.7, 87.9)
Routing:
- net +3.3V: track 8.47 -> 7.16 mm, vias 2 -> 1
Changed lines of the file:
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@@
 	(footprint "Capacitor_SMD:C_0603_1608Metric"
 		(layer "F.Cu")
-		(at 150.876 88.506 -90)
+		(at 150.749 87.884 -90)
 		(descr "Capacitor SMD 0603 (1608 Metric), square (rectangular) end terminal, IPC_7351 nominal, (Body size source: IPC-SM-782 page 76, https://www.pcb-3d.com/wordpress/wp-content/uploads/ipc-sm-782a_amendment_1_and_2.pdf), generated with kicad-footprint-generator")
 		(tags "capacitor")
@@
 	(footprint "AT2659:DFN150X100X80-6N"
 		(layer "F.Cu")
-		(at 152.781 88.549 90)
+		(at 152.654 87.927 90)
 		(property "Reference" "U3"
 			(at -1.989 0 360)
@@
 	)
 	(segment
-		(start 151.143 89.014)
-		(end 150.876 89.281)
-		(width 0.3)
-		(layer "F.Cu")
-		(net 4)
-	)
-	(segment
 		(start 151.298 93.629642)
 		(end 144.698 100.229642)
@@
 	)
 	(segment
-		(start 152.273 89.014)
-		(end 151.143 89.014)
+		(start 152.146 88.392)
+		(end 151.016 88.392)
 		(width 0.3)
 		(layer "F.Cu")
@@
 	)
 	(segment
-		(start 152.273 89.014)
-		(end 152.781 89.014)
+		(start 152.146 88.392)
+		(end 152.654 88.392)
 		(width 0.3)
 		(layer "F.Cu")
@@
 	)
 	(segment
-		(start 153.289 88.084)
-		(end 153.584 88.084)
-		(width 0.3)
-		(layer "F.Cu")
-		(net 5)
-	)
-	(segment
 		(start 152.398 102.968)
 		(end 152.398 100.813)
@@
 		(net 5)
 	)
-	(segment
-		(start 153.289 88.084)
-		(end 152.781 88.084)
-		(width 0.3)
-		(layer "F.Cu")
-		(net 5)
-	)
-	(segment
-		(start 153.584 88.084)
-		(end 153.924 87.744)
-		(width 0.3)
-		(layer "F.Cu")
-		(net 5)
-	)
 	(via
-		(at 153.924 87.744)
+		(at 153.797 87.122)
 		(size 0.6)
 		(drill 0.3)
@@
 		(net 5)
 	)
-	(via
-		(at 150.876 87.731)
-		(size 0.6)
-		(drill 0.3)
-		(layers "F.Cu" "B.Cu")
-		(net 5)
-	)
-	(segment
-		(start 153.924 87.744)
-		(end 150.889 87.744)
-		(width 0.3)
-		(layer "B.Cu")
-		(net 5)
-	)
 	(segment
-		(start 150.889 87.744)
-		(end 150.876 87.731)
+		(start 153.797 87.122)
+		(end 150.762 87.122)
 		(width 0.3)
 		(layer "B.Cu")
@@
 	)
 	(segment
-		(start 154.569 89.014)
-		(end 153.289 89.014)
+		(start 154.442 88.392)
+		(end 153.162 88.392)
 		(width 0.3)
 		(layer "F.Cu")
