File: PCB + Schematic/gpsBreakout/gpsBreakoutAutoroute.kicad_pcb (KiCad board)
At the start: 2 copper layers, 18.7 x 27.1 mm, 17 parts, among them J1 Header, U1 ATGM336H, U2 AT24CS32-STUM, U3 AT2659

Commit message: Finished board
Parts:
- moved R1 0.27 mm to (148.7, 103.2)
Routing:
- net +3.3V: track 57.1 -> 8.36 mm, vias 4 -> 2
- net VBAT: track 35.3 -> 0.00 mm, vias 2 -> 0
- net SDA: track 31.8 -> 0.00 mm, vias 1 -> 0
- net SCL: track 28.8 -> 0.00 mm, vias 1 -> 0
- net RESET: track 24.2 -> 0.00 mm, vias 1 -> 0
- net PPS: track 16.5 -> 0.00 mm, vias 3 -> 0
- net VCC_RF: track 9.19 -> 0.00 mm
- net TX: track 7.94 -> 0.00 mm, vias 2 -> 0
- net RX: track 5.61 -> 0.00 mm, vias 1 -> 0
- net RF: track 8.85 -> 7.78 mm
- net PASSIVE: track 6.13 -> 5.13 mm
- net Net-(AE2-FEED): track 2.06 -> 1.36 mm
- net GND: vias 4 -> 0
Other:
- board size 18.7 x 27.1 mm -> 17.9 x 26.7 mm
- board text removed: "Designed by Charles Nicholson, June 2024"
- board text removed: "GND"
- board text removed: "JLCJLCJLCJLC"
- board text removed: "JP1: 1 = passive, 3 = active"
- board text removed: "Made with support of Hack Club and NEWBS"
- board text removed: "PPS"
- board text removed: "RST"
- board text removed: "RX"
- board text removed: "SCL"
- board text removed: "SDA"
- board text removed: "TX"
- board text removed: "VCC"
- board text removed: "V_BAT"
- board text removed: "V_RF"
