File: PCB + Schematic/gpsBreakout/gpsBreakout.kicad_sch (KiCad schematic)
At the start: 10 parts, among them J1 Header, U1 ATGM336H, U2 AT24CS32-STUM

Commit message: Routing!
Parts:
- removed C1: 100 nF, symbol Device:C_Small
- added AE2: 1575AT43A0040001E, 1575AT43A0040E:ANT_1575AT_JOT-L, symbol Device:Antenna_Chip
- added BT1: MS621R, Battery:MS621R, symbol Device:Battery_Cell
- added C3, C5: 100 nF, Capacitor_SMD:C_0603_1608Metric, symbol Device:C_Small
- added C4: 470 pF, Capacitor_SMD:C_0402_1005Metric, symbol Device:C_Small
- added D1: SS14, Diode_SMD:D_SMA, symbol Device:D_Schottky_Small
- added L2: 6.8 nH, Inductor_SMD:L_0402_1005Metric, symbol Device:L_Small
- added U3: AT2659, AT2659:DFN150X100X80-6N, symbol RF_Amplifier:AT2659
- C2: footprint (none) -> Capacitor_SMD:C_0603_1608Metric; LCSC (none) -> C14663
- D2: footprint (none) -> LED_SMD:LED_0603_1608Metric; LCSC (none) -> C2286
- J1: footprint (none) -> Connector_PinHeader_2.54mm:PinHeader_1x10_P2.54mm_Vertical
- JP1: footprint (none) -> Jumper:SolderJumper-3_P1.3mm_Open_RoundedPad1.0x1.5mm
- L1: value 33nH -> 33 nH; footprint Inductor_SMD:L_0805_2012Metric_Pad1.15x1.40mm_HandSolder -> Inductor_SMD:L_0402_1005Metric; LCSC (none) -> C90178
- R1: footprint (none) -> Resistor_SMD:R_0402_1005Metric; LCSC (none) -> C25077
Connections:
- net +3.3V: now also C3.1, C5.1, D1.2 (A), U3.4 (VCC), U3.5 (SHDN)
- net ACTIVE: now also U3.6 (RF_OUT)
- net GND: now also AE1.2 (GND), AE2.2 (GND), BT1.2 (-), C3.2, C5.2, U3.1 (GND), U3.2 (GND)
- net VBAT: now also BT1.1 (+), D1.1 (K)
- new net: C4.2, L2.1
- new net: L2.2, U3.3 (RF_IN)
- new net: AE2.1 (FEED), C4.1

Commit message: Folding glider, plus some PCB stuff from later
Parts:
- AE1, AE2: symbol Device:Antenna_Chip -> symbols:Antenna_Chip
- BT1: symbol Device:Battery_Cell -> symbols:Battery_Cell
- C2, C3, C4, C5: symbol Device:C_Small -> symbols:C_Small
- D1: symbol Device:D_Schottky_Small -> symbols:D_Schottky_Small
- D2: symbol Device:LED_Small -> symbols:LED_Small
- J1: symbol Connector_Generic:Conn_01x10 -> symbols:Conn_01x10
- JP1: symbol Jumper:SolderJumper_3_Open -> symbols:SolderJumper_3_Open
- L1: symbol Device:L -> symbols:L
- L2: symbol Device:L_Small -> symbols:L_Small
- R1: symbol Device:R_Small -> symbols:R_Small
- U1: symbol RF_GPS:ATGM336H -> symbols:ATGM336H
- U2: symbol Memory_EEPROM:AT24CS32-STUM -> symbols:AT24CS32-STUM
- U3: symbol RF_Amplifier:AT2659 -> symbols:AT2659
Changed lines of the file:
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@@
 	)
 	(symbol
-		(lib_id "Device:C_Small")
+		(lib_id "symbols:C_Small")
 		(at 209.55 86.36 0)
 		(unit 1)
@@
 	)
 	(symbol
-		(lib_id "Device:Antenna_Chip")
+		(lib_id "symbols:Antenna_Chip")
 		(at 229.87 88.9 0)
 		(unit 1)
@@
 	)
 	(symbol
-		(lib_id "power:+3.3V")
+		(lib_id "symbols:+3.3V")
 		(at 194.31 139.7 0)
 		(unit 1)
@@
 	)
 	(symbol
-		(lib_id "Device:L_Small")
+		(lib_id "symbols:L_Small")
 		(at 214.63 55.88 0)
 		(unit 1)
@@
 	)
 	(symbol
-		(lib_id "power:GND")
+		(lib_id "symbols:GND")
 		(at 256.54 60.96 0)
 		(unit 1)
@@
 	)
 	(symbol
-		(lib_id "Device:LED_Small")
+		(lib_id "symbols:LED_Small")
 		(at 185.42 66.04 0)
 		(unit 1)
@@
 	)
 	(symbol
-		(lib_id "Connector_Generic:Conn_01x10")
+		(lib_id "symbols:Conn_01x10")
 		(at 176.53 132.08 180)
 		(unit 1)
@@
 	)
 	(symbol
-		(lib_id "Device:L")
+		(lib_id "symbols:L")
 		(at 241.3 97.79 90)
 		(unit 1)
@@
 	)
 	(symbol
-		(lib_id "Device:C_Small")
+		(lib_id "symbols:C_Small")
 		(at 214.63 50.8 0)
 		(unit 1)
@@
 	)
 	(symbol
-		(lib_id "power:+3.3V")
+		(lib_id "symbols:+3.3V")
 		(at 269.24 53.34 0)
 		(unit 1)
@@
 	(symbol
 		(lib_name "GND_15")
-		(lib_id "power:GND")
+		(lib_id "symbols:GND_15")
 		(at 210.82 48.26 0)
 		(unit 1)
@@
 	)
 	(symbol
-		(lib_id "power:GND")
+		(lib_id "symbols:GND")
 		(at 182.88 66.04 0)
 		(unit 1)
@@
 	)
 	(symbol
-		(lib_id "power:+3.3V")
+		(lib_id "symbols:+3.3V")
 		(at 166.37 102.87 0)
 		(unit 1)
@@
 	(symbol
 		(lib_name "GND_15")
-		(lib_id "power:GND")
+		(lib_id "symbols:GND_15")
 		(at 245.11 97.79 0)
 		(unit 1)
@@
 	)
 	(symbol
-		(lib_id "power:+3.3V")
+		(lib_id "symbols:+3.3V")
 		(at 189.23 78.74 0)
 		(unit 1)
@@
 	)
 	(symbol
-		(lib_id "power:GND")
+		(lib_id "symbols:GND")
 		(at 132.08 68.58 0)
 		(unit 1)
@@
 	)
 	(symbol
-		(lib_id "RF_GPS:ATGM336H")
+		(lib_id "symbols:ATGM336H")
 		(at 142.24 85.09 0)
 		(unit 1)
@@
 	)
 	(symbol
-		(lib_id "Device:C_Small")
+		(lib_id "symbols:C_Small")
 		(at 134.62 68.58 90)
 		(unit 1)
@@
 	)
 	(symbol
-		(lib_id "Memory_EEPROM:AT24CS32-STUM")
+		(lib_id "symbols:AT24CS32-STUM")
 		(at 189.23 86.36 0)
 		(unit 1)
@@
 	)
 	(symbol
-		(lib_id "Device:C_Small")
+		(lib_id "symbols:C_Small")
 		(at 256.54 58.42 0)
 		(unit 1)
@@
 	)
 	(symbol
-		(lib_id "Device:D_Schottky_Small")
+		(lib_id "symbols:D_Schottky_Small")
 		(at 144.78 135.89 0)
 		(unit 1)
@@
 	)
 	(symbol
-		(lib_id "power:GND")
+		(lib_id "symbols:GND")
 		(at 135.89 143.51 0)
 		(unit 1)
@@
 	)
 	(symbol
-		(lib_id "power:+3.3V")
+		(lib_id "symbols:+3.3V")
 		(at 142.24 68.58 0)
 		(unit 1)
@@
 	)
 	(symbol
-		(lib_id "power:+3.3V")
+		(lib_id "symbols:+3.3V")
 		(at 147.32 135.89 270)
 		(unit 1)
@@
 	)
 	(symbol
-		(lib_id "Device:Antenna_Chip")
+		(lib_id "symbols:Antenna_Chip")
 		(at 212.09 45.72 0)
 		(unit 1)
@@
 	(symbol
 		(lib_name "GND_15")
-		(lib_id "power:GND")
+		(lib_id "symbols:GND_15")
 		(at 229.87 91.44 0)
 		(unit 1)
@@
 	)
 	(symbol
-		(lib_id "Device:Battery_Cell")
+		(lib_id "symbols:Battery_Cell")
 		(at 135.89 140.97 0)
 		(unit 1)
@@
 	)
 	(symbol
-		(lib_id "RF_Amplifier:AT2659")
+		(lib_id "symbols:AT2659")
 		(at 246.38 44.45 0)
 		(unit 1)
@@
 	)
 	(symbol
-		(lib_id "power:GND")
+		(lib_id "symbols:GND")
 		(at 229.87 50.8 0)
 		(unit 1)
@@
 	)
 	(symbol
-		(lib_id "Jumper:SolderJumper_3_Open")
+		(lib_id "symbols:SolderJumper_3_Open")
 		(at 252.73 76.2 270)
 		(unit 1)
@@
 	)
 	(symbol
-		(lib_id "power:GND")
+		(lib_id "symbols:GND")
 		(at 139.7 115.57 0)
 		(unit 1)
@@
 	)
 	(symbol
-		(lib_id "power:GND")
+		(lib_id "symbols:GND")
 		(at 181.61 142.24 0)
 		(unit 1)
@@
 	)
 	(symbol
-		(lib_id "Device:R_Small")
+		(lib_id "symbols:R_Small")
 		(at 190.5 66.04 90)
 		(unit 1)
@@
 	)
 	(symbol
-		(lib_id "power:GND")
+		(lib_id "symbols:GND")
 		(at 189.23 93.98 0)
 		(unit 1)

Commit message: More work on the schematic
Parts:
- removed D1: SS14, Diode_SMD:D_SMA, symbol symbols:D_Schottky_Small
Other:
- moved on the sheet: BT1
Changed lines of the file:
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@@
 	(wire
 		(pts
-			(xy 135.89 135.89) (xy 142.24 135.89)
+			(xy 237.49 50.8) (xy 237.49 53.34)
 		)
 		(stroke
@@
 	(wire
 		(pts
-			(xy 237.49 50.8) (xy 237.49 53.34)
+			(xy 142.24 80.01) (xy 142.24 68.58)
 		)
 		(stroke
@@
 	(wire
 		(pts
-			(xy 142.24 80.01) (xy 142.24 68.58)
+			(xy 142.24 115.57) (xy 144.78 115.57)
 		)
 		(stroke
@@
 	(wire
 		(pts
-			(xy 142.24 115.57) (xy 144.78 115.57)
+			(xy 199.39 93.98) (xy 189.23 93.98)
 		)
 		(stroke
@@
 	(wire
 		(pts
-			(xy 199.39 93.98) (xy 189.23 93.98)
+			(xy 181.61 139.7) (xy 194.31 139.7)
 		)
 		(stroke
@@
 	(wire
 		(pts
-			(xy 181.61 139.7) (xy 194.31 139.7)
+			(xy 210.82 48.26) (xy 212.09 48.26)
 		)
 		(stroke
@@
 	(wire
 		(pts
-			(xy 210.82 48.26) (xy 212.09 48.26)
+			(xy 166.37 102.87) (xy 156.21 102.87)
 		)
 		(stroke
@@
 	(wire
 		(pts
-			(xy 166.37 102.87) (xy 156.21 102.87)
+			(xy 209.55 88.9) (xy 209.55 93.98)
 		)
 		(stroke
@@
 	(wire
 		(pts
-			(xy 209.55 88.9) (xy 209.55 93.98)
+			(xy 214.63 59.69) (xy 237.49 59.69)
 		)
 		(stroke
@@
 	(wire
 		(pts
-			(xy 214.63 59.69) (xy 237.49 59.69)
+			(xy 256.54 53.34) (xy 269.24 53.34)
 		)
 		(stroke
@@
 	(wire
 		(pts
-			(xy 256.54 53.34) (xy 269.24 53.34)
+			(xy 214.63 59.69) (xy 214.63 58.42)
 		)
 		(stroke
@@
 	(wire
 		(pts
-			(xy 214.63 59.69) (xy 214.63 58.42)
+			(xy 237.49 91.44) (xy 232.41 91.44)
 		)
 		(stroke
@@
 	(wire
 		(pts
-			(xy 237.49 91.44) (xy 232.41 91.44)
+			(xy 137.16 68.58) (xy 142.24 68.58)
 		)
 		(stroke
@@
 	(wire
 		(pts
-			(xy 137.16 68.58) (xy 142.24 68.58)
+			(xy 209.55 78.74) (xy 189.23 78.74)
 		)
 		(stroke
@@
 	(wire
 		(pts
-			(xy 209.55 78.74) (xy 189.23 78.74)
+			(xy 199.39 88.9) (xy 199.39 93.98)
 		)
 		(stroke
@@
 	(wire
 		(pts
-			(xy 199.39 88.9) (xy 199.39 93.98)
+			(xy 229.87 50.8) (xy 237.49 50.8)
 		)
 		(stroke
@@
 		)
 	)
-	(wire
-		(pts
-			(xy 229.87 50.8) (xy 237.49 50.8)
-		)
-		(stroke
-			(width 0)
-			(type default)
-		)
-	)
 	(global_label "RESET"
 		(shape input)
@@
 	(global_label "VBAT"
 		(shape input)
-		(at 135.89 135.89 180)
-		(fields_autoplaced yes)
-		(effects
-			(font
-				(size 1.27 1.27)
-			)
-			(justify right)
-		)
-		(property "Intersheetrefs" "${INTERSHEET_REFS}"
-			(at 128.49 135.89 0)
-			(effects
-				(font
-					(size 1.27 1.27)
-				)
-				(justify right)
+		(at 109.22 91.44 90)
+		(fields_autoplaced yes)
+		(effects
+			(font
+				(size 1.27 1.27)
+			)
+			(justify left)
+		)
+		(property "Intersheetrefs" "${INTERSHEET_REFS}"
+			(at 109.22 84.04 90)
+			(effects
+				(font
+					(size 1.27 1.27)
+				)
+				(justify left)
 				(hide yes)
 			)
@@
 	)
 	(symbol
-		(lib_id "symbols:D_Schottky_Small")
-		(at 144.78 135.89 0)
-		(unit 1)
-		(exclude_from_sim no)
-		(in_bom yes)
-		(on_board yes)
-		(dnp no)
-		(fields_autoplaced yes)
-		(property "Reference" "D1"
-			(at 144.526 129.54 0)
-			(effects
-				(font
-					(size 1.27 1.27)
-				)
-			)
-		)
-		(property "Value" "SS14"
-			(at 144.526 132.08 0)
-			(effects
-				(font
-					(size 1.27 1.27)
-				)
-			)
-		)
-		(property "Footprint" "Diode_SMD:D_SMA"
-			(at 144.78 135.89 90)
-			(effects
-				(font
-					(size 1.27 1.27)
-				)
-				(hide yes)
-			)
-		)
-		(property "Datasheet" "~"
-			(at 144.78 135.89 90)
-			(effects
-				(font
-					(size 1.27 1.27)
-				)
-				(hide yes)
-			)
-		)
-		(property "Description" "Schottky diode, small symbol"
-			(at 144.78 135.89 0)
-			(effects
-				(font
-					(size 1.27 1.27)
-				)
-				(hide yes)
-			)
-		)
-		(property "LCSC" "C2480"
-			(at 144.78 135.89 0)
-			(effects
-				(font
-					(size 1.27 1.27)
-				)
-				(hide yes)
-			)
-		)
-		(pin "2"
-		)
-		(pin "1"
-		)
-		(instances
-			(project "gpsBreakout"
-				(path "/f6412663-1207-425b-b708-3727894d909a"
-					(reference "D1")
-					(unit 1)
-				)
-			)
-		)
-	)
-	(symbol
 		(lib_id "symbols:GND")
-		(at 135.89 143.51 0)
+		(at 109.22 99.06 0)
 		(unit 1)
 		(exclude_from_sim no)
@@
 		(dnp no)
 		(property "Reference" "#PWR015"
-			(at 135.89 149.86 0)
+			(at 109.22 105.41 0)
 			(effects
 				(font
@@
 		)
 		(property "Value" "GND"
-			(at 135.89 147.32 0)
+			(at 109.22 102.87 0)
 			(effects
 				(font
@@
 		)
 		(property "Footprint" ""
-			(at 135.89 143.51 0)
+			(at 109.22 99.06 0)
 			(effects
 				(font
@@
 		)
 		(property "Datasheet" ""
-			(at 135.89 143.51 0)
+			(at 109.22 99.06 0)
 			(effects
 				(font
@@
 		)
 		(property "Description" "Power symbol creates a global label with name \"GND\" , ground"
-			(at 135.89 143.51 0)
+			(at 109.22 99.06 0)
 			(effects
 				(font
@@
 				(path "/f6412663-1207-425b-b708-3727894d909a"
 					(reference "#PWR07")
-					(unit 1)
-				)
-			)
-		)
-	)
-	(symbol
-		(lib_id "symbols:+3.3V")
-		(at 147.32 135.89 270)
-		(unit 1)
-		(exclude_from_sim no)
-		(in_bom yes)
-		(on_board yes)
-		(dnp no)
-		(fields_autoplaced yes)
-		(property "Reference" "#PWR014"
-			(at 143.51 135.89 0)
-			(effects
-				(font
-					(size 1.27 1.27)
-				)
-				(hide yes)
-			)
-		)
-		(property "Value" "+3.3V"
-			(at 151.13 135.8899 90)
-			(effects
-				(font
-					(size 1.27 1.27)
-				)
-				(justify left)
-			)
-		)
-		(property "Footprint" ""
-			(at 147.32 135.89 0)
-			(effects
-				(font
-					(size 1.27 1.27)
-				)
-				(hide yes)
-			)
-		)
-		(property "Datasheet" ""
-			(at 147.32 135.89 0)
-			(effects
-				(font
-					(size 1.27 1.27)
-				)
-				(hide yes)
-			)
-		)
-		(property "Description" "Power symbol creates a global label with name \"+3.3V\""
-			(at 147.32 135.89 0)
-			(effects
-				(font
-					(size 1.27 1.27)
-				)
-				(hide yes)
-			)
-		)
-		(pin "1"
-		)
-		(instances
-			(project "gpsBreakout"
-				(path "/f6412663-1207-425b-b708-3727894d909a"
-					(reference "#PWR014")
 					(unit 1)
 				)
@@
 	(symbol
 		(lib_id "symbols:Battery_Cell")
-		(at 135.89 140.97 0)
+		(at 109.22 96.52 0)
 		(unit 1)
 		(exclude_from_sim no)
@@
 		(dnp no)
 		(property "Reference" "BT1"
-			(at 138.43 138.43 0)
+			(at 111.76 93.98 0)
 			(effects
 				(font
@@
 		)
 		(property "Value" "MS621R"
-			(at 138.43 140.97 0)
+			(at 111.76 96.52 0)
 			(effects
 				(font
@@
 		)
 		(property "Footprint" "Battery:MS621R"
-			(at 135.89 139.446 90)
+			(at 109.22 94.996 90)
 			(effects
 				(font
@@
 		)
 		(property "Datasheet" "~"
-			(at 135.89 139.446 90)
+			(at 109.22 94.996 90)
 			(effects
 				(font
@@
 		)
 		(property "Description" "Single-cell battery"
-			(at 135.89 140.97 0)
-			(effects
-				(font
+			(at 109.22 96.52 0)
+			(effects
+				(font

Commit message: Finished PCB
Parts:
- AE1, AE2: footprint 1575AT43A0040E:ANT_1575AT_JOT-L -> footprints:ANT_1575AT_JOT-L
- BT1: footprint Battery:MS621R -> footprints:MS621R
- C2, C3, C5: footprint Capacitor_SMD:C_0603_1608Metric -> footprints:C_0603_1608Metric
- C4: footprint Capacitor_SMD:C_0402_1005Metric -> footprints:C_0402_1005Metric
- D2: footprint LED_SMD:LED_0603_1608Metric -> footprints:LED_0603_1608Metric
- J1: footprint Connector_PinHeader_2.54mm:PinHeader_1x10_P2.54mm_Vertical -> footprints:PinHeader_1x10_P2.54mm_Vertical
- JP1: footprint Jumper:SolderJumper-3_P1.3mm_Open_RoundedPad1.0x1.5mm -> footprints:SolderJumper-3_P1.3mm_Open_RoundedPad1.0x1.5mm
- L1, L2: footprint Inductor_SMD:L_0402_1005Metric -> footprints:L_0402_1005Metric
- R1: footprint Resistor_SMD:R_0402_1005Metric -> footprints:R_0402_1005Metric
- U1: footprint RF_GPS:ATGM336H -> footprints:ATGM336H
- U2: footprint Package_TO_SOT_SMD:SOT-23-5 -> footprints:SOT-23-5
- U3: footprint AT2659:DFN150X100X80-6N -> footprints:DFN150X100X80-6N
Changed lines of the file:
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@@
 			)
 		)
-		(property "Footprint" "Capacitor_SMD:C_0603_1608Metric"
+		(property "Footprint" "footprints:C_0603_1608Metric"
 			(at 209.55 86.36 0)
 			(effects
@@
 			)
 		)
-		(property "Footprint" "1575AT43A0040E:ANT_1575AT_JOT-L"
+		(property "Footprint" "footprints:ANT_1575AT_JOT-L"
 			(at 227.33 84.455 0)
 			(effects
@@
 			)
 		)
-		(property "Footprint" "Inductor_SMD:L_0402_1005Metric"
+		(property "Footprint" "footprints:L_0402_1005Metric"
 			(at 214.63 55.88 0)
 			(effects
@@
 			)
 		)
-		(property "Footprint" "LED_SMD:LED_0603_1608Metric"
+		(property "Footprint" "footprints:LED_0603_1608Metric"
 			(at 185.42 66.04 90)
 			(effects
@@
 			)
 		)
-		(property "Footprint" "Connector_PinHeader_2.54mm:PinHeader_1x10_P2.54mm_Vertical"
+		(property "Footprint" "footprints:PinHeader_1x10_P2.54mm_Vertical"
 			(at 176.53 132.08 0)
 			(effects
@@
 			)
 		)
-		(property "Footprint" "Inductor_SMD:L_0402_1005Metric"
+		(property "Footprint" "footprints:L_0402_1005Metric"
 			(at 241.3 97.79 0)
 			(effects
@@
 			)
 		)
-		(property "Footprint" "Capacitor_SMD:C_0402_1005Metric"
+		(property "Footprint" "footprints:C_0402_1005Metric"
 			(at 214.63 50.8 0)
 			(effects
@@
 			)
 		)
-		(property "Footprint" "RF_GPS:ATGM336H"
+		(property "Footprint" "footprints:ATGM336H"
 			(at 142.24 85.09 0)
 			(effects
@@
 			)
 		)
-		(property "Footprint" "Capacitor_SMD:C_0603_1608Metric"
+		(property "Footprint" "footprints:C_0603_1608Metric"
 			(at 134.62 68.58 0)
 			(effects
@@
 			)
 		)
-		(property "Footprint" "Package_TO_SOT_SMD:SOT-23-5"
+		(property "Footprint" "footprints:SOT-23-5"
 			(at 189.23 86.36 0)
 			(effects
@@
 			)
 		)
-		(property "Footprint" "Capacitor_SMD:C_0603_1608Metric"
+		(property "Footprint" "footprints:C_0603_1608Metric"
 			(at 256.54 58.42 0)
 			(effects
@@
 			)
 		)
-		(property "Footprint" "1575AT43A0040E:ANT_1575AT_JOT-L"
+		(property "Footprint" "footprints:ANT_1575AT_JOT-L"
 			(at 209.55 41.275 0)
 			(effects
@@
 			)
 		)
-		(property "Footprint" "Battery:MS621R"
+		(property "Footprint" "footprints:MS621R"
 			(at 109.22 94.996 90)
 			(effects
@@
 			)
 		)
-		(property "Footprint" "AT2659:DFN150X100X80-6N"
+		(property "Footprint" "footprints:DFN150X100X80-6N"
 			(at 246.38 44.45 0)
 			(effects
@@
 			)
 		)
-		(property "Footprint" "Jumper:SolderJumper-3_P1.3mm_Open_RoundedPad1.0x1.5mm"
+		(property "Footprint" "footprints:SolderJumper-3_P1.3mm_Open_RoundedPad1.0x1.5mm"
 			(at 252.73 76.2 0)
 			(effects
@@
 			)
 		)
-		(property "Footprint" "Resistor_SMD:R_0402_1005Metric"
+		(property "Footprint" "footprints:R_0402_1005Metric"
 			(at 190.5 66.04 0)
 			(effects

Commit message: Actually finished board for real?
Parts:
- added R2, R3: 1.8 K, Resistor_SMD:R_0603_1608Metric, symbol symbols:R_Small
Connections:
- net +3.3V: now also R2.1, R3.1
- net SCL: now also R3.2
- net SDA: now also R2.2

Commit message: Actually finished board, did GPS work
Parts:
- removed J1: Header, footprints:PinHeader_1x10_P2.54mm_Vertical, symbol symbols:Conn_01x10
- removed R1: 1 K, footprints:R_0402_1005Metric, symbol symbols:R_Small
- added J2: Header, Connector_PinHeader_2.54mm:PinHeader_1x11_P2.54mm_Vertical, symbol Connector_Generic:Conn_01x11
- added R7: 1 K, Resistor_SMD:R_0402_1005Metric, symbol symbols:R_Small
- D2: value RED -> YELLOW; footprint footprints:LED_0603_1608Metric -> LED_SMD:LED_0603_1608Metric; LCSC C2286 -> C72038
- U2: value AT24CS32-STUM -> BL24C32F-RRRC; footprint footprints:SOT-23-5 -> Package_TO_SOT_SMD:SOT-23-5; LCSC (none) -> C5185883
Connections:
- net +3.3V: now also J2.2 (Pin_2); no longer U1.5 (EN)
- net GND: now also J2.1 (Pin_1)
- net PPS: now also J2.6 (Pin_6), R7.2
- net RESET: now also J2.5 (Pin_5)
- net RX: now also J2.10 (Pin_10)
- net SCL: now also J2.7 (Pin_7)
- net SDA: now also J2.8 (Pin_8)
- net TX: now also J2.9 (Pin_9)
- net VCC_RF: now also J2.4 (Pin_4)
- net at D2.2 (A): now also R7.1
- net VBAT renamed V_BAT
- net V_BAT: now also J2.3 (Pin_3)
- new net GPS_EN: J2.11 (Pin_11), U1.5 (EN)

Commit message: More gps work
Parts:
- AE1, AE2: value 1575AT43A0040001E -> GPS1003; footprint footprints:ANT_1575AT_JOT-L -> RF_Antenna:GPS1003
- L2: LCSC C90136 -> C84403
- U1: LCSC C5117921 -> C90770
Changed lines of the file:
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@@
-	)
-	(symbol
-		(lib_id "symbols:Antenna_Chip")
-		(at 229.87 88.9 0)
-		(unit 1)
-		(exclude_from_sim no)
-		(in_bom yes)
-		(on_board yes)
-		(dnp no)
-		(fields_autoplaced yes)
-		(property "Reference" "AE1"
-			(at 234.95 85.0899 0)
-			(effects
-				(font
-					(size 1.27 1.27)
-				)
-				(justify left)
-			)
-		)
-		(property "Value" "1575AT43A0040001E"
-			(at 234.95 87.6299 0)
-			(effects
-				(font
-					(size 1.27 1.27)
-				)
-				(justify left)
-			)
-		)
-		(property "Footprint" "footprints:ANT_1575AT_JOT-L"
-			(at 227.33 84.455 0)
-			(effects
-				(font
-					(size 1.27 1.27)
-				)
-				(hide yes)
-			)
-		)
-		(property "Datasheet" "~"
-			(at 227.33 84.455 0)
-			(effects
-				(font
-					(size 1.27 1.27)
-				)
-				(hide yes)
-			)
-		)
-		(property "Description" "Ceramic chip antenna with pin for PCB trace"
-			(at 229.87 88.9 0)
-			(effects
-				(font
-					(size 1.27 1.27)
-				)
-				(hide yes)
-			)
-		)
-		(pin "1"
-		)
-		(pin "2"
-		)
-		(instances
-			(project "gpsBreakout"
-				(path "/f6412663-1207-425b-b708-3727894d909a"
-					(reference "AE1")
-					(unit 1)
-				)
-			)
-		)
 	)
 	(symbol
@@
 			)
 		)
-		(property "LCSC" "C90136"
+		(property "LCSC" "C84403"
 			(at 214.63 55.88 0)
 			(effects
@@
 	)
 	(symbol
+		(lib_id "symbols:Antenna_Chip")
+		(at 229.87 88.9 0)
+		(unit 1)
+		(exclude_from_sim no)
+		(in_bom yes)
+		(on_board yes)
+		(dnp no)
+		(fields_autoplaced yes)
+		(property "Reference" "AE1"
+			(at 234.95 85.0899 0)
+			(effects
+				(font
+					(size 1.27 1.27)
+				)
+				(justify left)
+			)
+		)
+		(property "Value" "GPS1003"
+			(at 234.95 87.6299 0)
+			(effects
+				(font
+					(size 1.27 1.27)
+				)
+				(justify left)
+			)
+		)
+		(property "Footprint" "RF_Antenna:GPS1003"
+			(at 227.33 84.455 0)
+			(effects
+				(font
+					(size 1.27 1.27)
+				)
+				(hide yes)
+			)
+		)
+		(property "Datasheet" "~"
+			(at 227.33 84.455 0)
+			(effects
+				(font
+					(size 1.27 1.27)
+				)
+				(hide yes)
+			)
+		)
+		(property "Description" "Ceramic chip antenna with pin for PCB trace"
+			(at 229.87 88.9 0)
+			(effects
+				(font
+					(size 1.27 1.27)
+				)
+				(hide yes)
+			)
+		)
+		(pin "1"
+		)
+		(pin "2"
+		)
+		(instances
+			(project "gpsBreakout"
+				(path "/f6412663-1207-425b-b708-3727894d909a"
+					(reference "AE1")
+					(unit 1)
+				)
+			)
+		)
+	)
+	(symbol
 		(lib_id "symbols:GND")
 		(at 132.08 68.58 0)
@@
 			)
 		)
-		(property "LCSC" "C5117921"
+		(property "LCSC" "C90770"
 			(at 142.24 85.09 0)
 			(effects
@@
 			)
 		)
-		(property "Value" "1575AT43A0040001E"
+		(property "Value" "GPS1003"
 			(at 217.17 44.4499 0)
 			(effects
@@
 			)
 		)
-		(property "Footprint" "footprints:ANT_1575AT_JOT-L"
+		(property "Footprint" "RF_Antenna:GPS1003"
 			(at 209.55 41.275 0)
 			(effects
