File: PCB + Schematic/StratoSoar-MK3.0/StratoSoar-MK3.0.kicad_sch (KiCad schematic)
At the start: 82 parts, among them J1 Power, J11 Signal, J12 Rudder, J2 Battery, J3 USB-C, J4 J Link, J5 Antenna, J6 Rudder, J8 Button, Q1 DMN1019USN-13, Q2 DMN1019USN-13, Q7 BSS138, Q8 BSS138, Q9 BSS138, SW1 RESET, SW2 PWR_SW, SW5 EEPROM, U1 Ra-01, U10 ICM-20948, U11 DSK321STD, U12 XC6206P332MR-G, U2 ATSAMD21G18A-A, U4 ATGM336H, U5 BME280, U6 AT24C512C-SSHD-T, U7 AT24CS32-STUM, U9 CJ6206B18M

Commit message: Basic layout
Parts:
- added C15: 100 nF, Capacitor_SMD:C_0402_1005Metric, symbol symbols:C_Small
- C4: footprint Capacitor_SMD:C_0402_1005Metric -> Capacitor_SMD:C_0603_1608Metric
- C7: footprint Capacitor_SMD:C_0603_1608Metric -> Capacitor_SMD:C_0402_1005Metric; LCSC C15849 -> C52923
Connections:
- net GND: now also C15.1
- net GPS_SCL: now also U7.1 (SCL)
- net GPS_SDA: no longer U7.1 (SCL)
- net at SW5.2 (B), U6.8 (VCC): now also C15.2
Changed lines of the file:
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@@
 	)
 	(junction
+		(at 157.48 92.71)
+		(diameter 0)
+		(color 0 0 0 0)
+	)
+	(junction
 		(at 355.6 215.9)
 		(diameter 0)
@@
 	(wire
 		(pts
+			(xy 153.67 97.79) (xy 157.48 97.79)
+		)
+		(stroke
+			(width 0)
+			(type default)
+		)
+	)
+	(wire
+		(pts
 			(xy 85.09 185.42) (xy 85.09 187.96)
 		)
@@
 	(wire
 		(pts
+			(xy 157.48 97.79) (xy 157.48 92.71)
+		)
+		(stroke
+			(width 0)
+			(type default)
+		)
+	)
+	(wire
+		(pts
 			(xy 133.35 260.35) (xy 137.16 260.35)
 		)
@@
 		)
 	)
-	(global_label "GPS_SDA"
+	(global_label "GPS_SCL"
 		(shape input)
 		(at 370.84 86.36 0)
@@
 		)
 		(property "Intersheetrefs" "${INTERSHEET_REFS}"
-			(at 382.1104 86.36 0)
+			(at 382.0499 86.36 0)
 			(effects
 				(font
@@
 	)
 	(symbol
+		(lib_name "GND_15")
+		(lib_id "power:GND")
+		(at 148.59 97.79 0)
+		(unit 1)
+		(exclude_from_sim no)
+		(in_bom yes)
+		(on_board yes)
+		(dnp no)
+		(property "Reference" "#PWR034"
+			(at 148.59 104.14 0)
+			(effects
+				(font
+					(size 1.27 1.27)
+				)
+				(hide yes)
+			)
+		)
+		(property "Value" "GND"
+			(at 148.59 102.235 0)
+			(effects
+				(font
+					(size 1.27 1.27)
+				)
+			)
+		)
+		(property "Footprint" ""
+			(at 148.59 97.79 0)
+			(effects
+				(font
+					(size 1.27 1.27)
+				)
+				(hide yes)
+			)
+		)
+		(property "Datasheet" ""
+			(at 148.59 97.79 0)
+			(effects
+				(font
+					(size 1.27 1.27)
+				)
+				(hide yes)
+			)
+		)
+		(property "Description" ""
+			(at 148.59 97.79 0)
+			(effects
+				(font
+					(size 1.27 1.27)
+				)
+				(hide yes)
+			)
+		)
+		(pin "1"
+		)
+		(instances
+			(project "StratoSoar-MK3.0"
+				(path "/a5ed86dc-e941-4edd-8d1d-eae06db8d6f6"
+					(reference "#PWR034")
+					(unit 1)
+				)
+			)
+		)
+	)
+	(symbol
 		(lib_id "symbols:GND")
 		(at 369.57 68.58 0)
@@
 	)
 	(symbol
+		(lib_id "symbols:C_Small")
+		(at 151.13 97.79 90)
+		(unit 1)
+		(exclude_from_sim no)
+		(in_bom yes)
+		(on_board yes)
+		(dnp no)
+		(fields_autoplaced yes)
+		(property "Reference" "C15"
+			(at 151.1363 91.44 90)
+			(effects
+				(font
+					(size 1.27 1.27)
+				)
+			)
+		)
+		(property "Value" "100 nF"
+			(at 151.1363 93.98 90)
+			(effects
+				(font
+					(size 1.27 1.27)
+				)
+			)
+		)
+		(property "Footprint" "Capacitor_SMD:C_0402_1005Metric"
+			(at 151.13 97.79 0)
+			(effects
+				(font
+					(size 1.27 1.27)
+				)
+				(hide yes)
+			)
+		)
+		(property "Datasheet" "~"
+			(at 151.13 97.79 0)
+			(effects
+				(font
+					(size 1.27 1.27)
+				)
+				(hide yes)
+			)
+		)
+		(property "Description" "Unpolarized capacitor, small symbol"
+			(at 151.13 97.79 0)
+			(effects
+				(font
+					(size 1.27 1.27)
+				)
+				(hide yes)
+			)
+		)
+		(property "LCSC" "C1525"
+			(at 151.13 97.79 0)
+			(effects
+				(font
+					(size 1.27 1.27)
+				)
+				(hide yes)
+			)
+		)
+		(pin "1"
+		)
+		(pin "2"
+		)
+		(instances
+			(project "StratoSoar-MK3.0"
+				(path "/a5ed86dc-e941-4edd-8d1d-eae06db8d6f6"
+					(reference "C15")
+					(unit 1)
+				)
+			)
+		)
+	)
+	(symbol
 		(lib_id "Transistor_FET:DMN1019USN-13")
 		(at 347.98 171.45 90)
@@
 			)
 		)
-		(property "Footprint" "Capacitor_SMD:C_0603_1608Metric"
+		(property "Footprint" "Capacitor_SMD:C_0402_1005Metric"
 			(at 34.29 172.72 0)
 			(effects
@@
 			)
 		)
-		(property "LCSC" "C15849"
+		(property "LCSC" "C52923"
 			(at 34.29 172.72 90)
 			(effects
@@
 			)
 		)
-		(property "Footprint" "Capacitor_SMD:C_0402_1005Metric"
+		(property "Footprint" "Capacitor_SMD:C_0603_1608Metric"
 			(at 149.86 160.02 0)
 			(effects

Commit message: IMU work
Other:
- note added: "DOES THE IMU HAVE BUILT IN I2C PULLUP RESISTORS"
- note removed: "EDIT IMU 10 K RESISTORS"
Changed lines of the file:
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@@
+		)
+	)
+	(text "DOES THE IMU HAVE BUILT IN I2C PULLUP RESISTORS"
+		(exclude_from_sim no)
+		(at 243.84 128.905 0)
+		(effects
+			(font
+				(size 5 5)
+				(thickness 1)
+				(bold yes)
+			)
 		)
 	)
@@
 			)
 		)
-	)
-	(text "EDIT IMU 10 K RESISTORS"
-		(exclude_from_sim no)
-		(at 226.06 132.715 0)
-		(effects
-			(font
-				(size 5 5)
-			)
-		)
