File: PCB + Schematic/imuBreakout/imuBreakout.kicad_pcb (KiCad board)
At the start: 2 copper layers, 15.8 x 16.8 mm, 18 parts, among them J1 Header, Q1 BSS138, Q2 BSS138, Q3 BSS138, U1 ICM-20948, U2 CJ6206B18M

Commit message: IMU work
Parts:
- removed R7: 10 K, Resistor_SMD:R_0402_1005Metric
- added R4: 10 K, Resistor_SMD:R_0402_1005Metric, F.Cu at (160.1, 96.8)
- renumbered C6 to C1, C3 to C2, C2 to C3, C1 to C4, R4 to R1, R1 to R2, R2 to R5, R5 to R6

Commit message: GPS, IMU
Other:
- board text added: "JLCJLCJLCJLC"
Changed lines of the file:
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@@
 			)
 		)
-		(property "LCSC" "C15849"
+		(property "LCSC" "C52923"
 			(at 0 0 -90)
 			(unlocked yes)
@@
 			)
 		)
-		(property "LCSC" "C15849"
+		(property "LCSC" "C52923"
 			(at 0 0 0)
 			(unlocked yes)
@@
 			)
 			(justify left bottom mirror)
+		)
+	)
+	(gr_text "JLCJLCJLCJLC"
+		(at 151.003 84.455 90)
+		(layer "B.SilkS")
+		(effects
+			(font
+				(size 1 1)
+				(thickness 0.15)
+			)
+			(justify left bottom mirror)
