File: PCB + Schematic/imuBreakout/imuBreakout.kicad_sch (KiCad schematic)
At the start: 17 parts, among them J1 Header, Q1 BSS138, Q2 BSS138, Q3 BSS138, U1 ICM-20948, U2 CJ6206B18M

Commit message: IMU stuff
Parts:
- J1: footprint (none) -> Connector_PinHeader_2.54mm:PinHeader_1x05_P2.54mm_Vertical
- Q1, Q2, Q3: LCSC (none) -> C5224268
- U1: LCSC (none) -> C726001
Changed lines of the file:
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@@
+			)
+		)
+		(property "LCSC" "C5224268"
+			(at 218.44 123.19 90)
+			(effects
+				(font
+					(size 1.27 1.27)
+				)
+				(hide yes)
 			)
 		)
@@
 			)
 		)
+		(property "LCSC" "C726001"
+			(at 154.94 105.41 0)
+			(effects
+				(font
+					(size 1.27 1.27)
+				)
+				(hide yes)
+			)
+		)
 		(pin "24"
 		)
@@
 			)
 		)
-		(property "Footprint" ""
+		(property "Footprint" "Connector_PinHeader_2.54mm:PinHeader_1x05_P2.54mm_Vertical"
 			(at 181.61 55.88 0)
 			(effects
@@
 			)
 		)
+		(property "LCSC" "C5224268"
+			(at 218.44 146.05 90)
+			(effects
+				(font
+					(size 1.27 1.27)
+				)
+				(hide yes)
+			)
+		)
 		(pin "1"
 		)
@@
 			(effects
 				(font
+					(size 1.27 1.27)
+				)
+				(hide yes)
+			)
+		)
+		(property "LCSC" "C5224268"
+			(at 218.44 100.33 90)
+			(effects
+				(font

Commit message: IMU work
Parts:
- removed R7: 10 K, Resistor_SMD:R_0402_1005Metric, symbol symbols:R_Small
- added R6: 10 K, Resistor_SMD:R_0402_1005Metric, symbol symbols:R_Small
- R1, R2, R3, R4, R5: LCSC C25077 -> C25744
- renumbered C6 to C1, C3 to C2, C2 to C3, C1 to C4
Connections:
- net +1V8: now also R2.1; no longer R4.1
- net INTH: now also R6.2; no longer R5.2
- net INTL: now also R1.2; no longer R4.2
- net SCLH: now also R4.2
- net SDAH: now also R5.2; no longer R2.2
- net SDAL: now also R2.2; no longer R1.2
- net VCC: now also R4.1, R6.1; no longer R2.1

Commit message: GPS, IMU
Parts:
- C4, C5: LCSC C15849 -> C52923
Changed lines of the file:
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@@
 			)
 		)
-		(property "LCSC" "C15849"
+		(property "LCSC" "C52923"
 			(at 205.74 73.66 0)
 			(effects
@@
 			)
 		)
-		(property "LCSC" "C15849"
+		(property "LCSC" "C52923"
 			(at 228.6 73.66 0)
 			(effects
