File: PCB + Schematic/loRa/loRa.kicad_sch (KiCad schematic)
At the start: 15 parts, among them J1 Analog, J10 Right, J11 Left, J12 Right, J13 OLED, J2 Digital, J3 Left, J4 Right, J5 GPS, J6 MPU-9250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

Commit message: LoRa PCB and case
Parts:
- removed J1: Analog, Connector_PinHeader_2.54mm:PinHeader_1x15_P2.54mm_Vertical, symbol Connector_Generic:Conn_01x15
- removed J10, J12, J7: Right, symbol Connector_Generic:Conn_01x06
- removed J11, J8, J9: Left, symbol Connector_Generic:Conn_01x06
- removed J13: OLED, symbol Connector_Generic:Conn_01x04
- removed J2: Digital, Connector_PinHeader_2.54mm:PinHeader_1x15_P2.54mm_Vertical, symbol Connector_Generic:Conn_01x15
- removed J3: Left, symbol Connector_Generic:Conn_01x08
- removed J4: Right, symbol Connector_Generic:Conn_01x08
- removed J5: GPS, symbol Connector_Generic:Conn_01x05
- removed J6: MPU-9250, symbol Connector_Generic:Conn_01x10
- added BT1: 3V, Battery:BatteryHolder_Keystone_2462_2xAA, symbol Device:Battery
- added H1, H2, H3, H4: MountingHole, MountingHole:MountingHole_3.2mm_M3, symbol Mechanical:MountingHole
- added J1: Left, Connector_PinHeader_2.54mm:PinHeader_1x08_P2.54mm_Vertical, symbol Connector_Generic:Conn_01x08
- added J2: Right, Connector_PinHeader_2.54mm:PinHeader_1x08_P2.54mm_Vertical, symbol Connector_Generic:Conn_01x08
- added J3: GPS, Connector_PinHeader_2.54mm:PinHeader_1x05_P2.54mm_Vertical, symbol Connector_Generic:Conn_01x05
- added J4: MPU-9250, Connector_PinHeader_2.54mm:PinHeader_1x10_P2.54mm_Vertical, symbol Connector_Generic:Conn_01x10
- added J7: OLED, Connector_PinHeader_2.54mm:PinHeader_1x04_P2.54mm_Vertical, symbol Connector_Generic:Conn_01x04
- added R2: 1.8 K, Resistor_THT:R_Axial_DIN0207_L6.3mm_D2.5mm_P7.62mm_Horizontal, symbol Device:R_Small
- added R3: 1 K, Resistor_THT:R_Axial_DIN0207_L6.3mm_D2.5mm_P7.62mm_Horizontal, symbol Device:R_Small
- added SW1: SW_SPDT, Button_Switch_THT:SW_Slide_SPDT, symbol Switch:SW_SPDT
- added U1: ESP32-DEVKIT-V1, ESP32-DEVKIT-V1:MODULE_ESP32_DEVKIT_V1, symbol ESP32-DEVKIT-V1:ESP32-DEVKIT-V1
- D1: footprint (none) -> LED_THT:LED_D3.0mm
- R1: value 220 -> 1.8 K; footprint (none) -> Resistor_THT:R_Axial_DIN0207_L6.3mm_D2.5mm_P7.62mm_Horizontal
Connections:
- net +3.3V: now also J1.3 (Pin_3), J3.1 (Pin_1), J4.1 (Pin_1), J7.2 (Pin_2), U1.1 (3V3)
- net CS: now also J2.2 (Pin_2), U1.4 (D2)
- net DIO0: now also J1.5 (Pin_5), U1.26 (D14)
- net DIO1: now also J1.6 (Pin_6)
- net DIO2: now also J1.7 (Pin_7)
- net DIO3: now also J1.8 (Pin_8)
- net DIO4: now also J2.7 (Pin_7)
- net DIO5: now also J2.6 (Pin_6)
- net GND: now also R1.2, J1.1 (Pin_1), J1.2 (Pin_2), J2.1 (Pin_1), J2.8 (Pin_8), J3.2 (Pin_2), J4.2 (Pin_2), J7.1 (Pin_1), R2.2, SW1.1 (A), U1.2 (GND), U1.29 (GND)
- net LED: now also R3.1, U1.28 (D13); no longer R1.2
- net LORA_RST: now also J1.4 (Pin_4), U1.27 (D12)
- net MISO: now also J2.4 (Pin_4), U1.10 (D19)
- net MOSI: now also J2.3 (Pin_3), U1.23 (D25)
- net RX: now also J3.4 (Pin_4), U1.6 (RX2)
- net SCK: now also J2.5 (Pin_5), U1.9 (D18)
- net SCL: now also J4.3 (Pin_3), J7.3 (Pin_3), R2.1, U1.14 (D22)
- net SDA: now also R1.1, J4.4 (Pin_4), J7.4 (Pin_4), U1.11 (D21)
- net TX: now also J3.3 (Pin_3), U1.7 (TX2)
- net at D1.2 (A): now also R3.2; no longer R1.1
- new net: BT1.2 (-), SW1.2 (B)
- new net +BATT: BT1.1 (+), U1.30 (VIN)
