File: PCB + Schematic/loRa/loRa.kicad_pcb (KiCad board)
At the start: 2 copper layers, 43.2 x 17.8 mm, 6 parts, among them J1 Analog, J2 Digital

Commit message: LoRa PCB and case
Parts:
- removed MH1, MH2, MH3, MH4: MountingHole_65mil, Arduino_MountingHole:MountingHole_65mil
- added BT1: 3V, Battery:BatteryHolder_Keystone_2462_2xAA, B.Cu at (193.6, 133.2)
- added D1: RED, LED_THT:LED_D3.0mm, F.Cu at (246.5, 106.4)
- added G***: LOGO, LOGO, F.Cu at (207.4, 126.1)
- added G***: LOGO, LOGO, F.Cu at (234.1, 118.1)
- added H1: MountingHole, MountingHole:MountingHole_3.2mm_M3, F.Cu at (247.8, 84.7)
- added H2: MountingHole, MountingHole:MountingHole_3.2mm_M3, F.Cu at (238.1, 132.3)
- added H3: MountingHole, MountingHole:MountingHole_3.2mm_M3, F.Cu at (188.2, 139.6)
- added H4: MountingHole, MountingHole:MountingHole_3.2mm_M3, F.Cu at (188.0, 84.7)
- added J3: GPS, Connector_PinHeader_2.54mm:PinHeader_1x05_P2.54mm_Vertical, F.Cu at (232.4, 99.8)
- added J4: MPU-9250, Connector_PinHeader_2.54mm:PinHeader_1x10_P2.54mm_Vertical, B.Cu at (245.1, 96.6)
- added J7: OLED, Connector_PinHeader_2.54mm:PinHeader_1x04_P2.54mm_Vertical, F.Cu at (209.2, 108.8)
- added R1: 1.8 K, Resistor_THT:R_Axial_DIN0207_L6.3mm_D2.5mm_P7.62mm_Horizontal, F.Cu at (222.8, 92.8)
- added R2: 1.8 K, Resistor_THT:R_Axial_DIN0207_L6.3mm_D2.5mm_P7.62mm_Horizontal, F.Cu at (227.6, 92.8)
- added R3: 1 K, Resistor_THT:R_Axial_DIN0207_L6.3mm_D2.5mm_P7.62mm_Horizontal, F.Cu at (233.0, 106.4)
- added SW1: SW_SPDT, Button_Switch_THT:SW_Slide_SPDT, F.Cu at (225.7, 106.3)
- added U1: ESP32-DEVKIT-V1, ESP32-DEVKIT-V1:MODULE_ESP32_DEVKIT_V1, F.Cu at (224.3, 125.7)
- J1: value Analog -> Left; footprint Connector_PinHeader_2.54mm:PinHeader_1x15_P2.54mm_Vertical -> Connector_PinHeader_2.54mm:PinHeader_1x08_P2.54mm_Vertical
- J2: value Digital -> Right; footprint Connector_PinHeader_2.54mm:PinHeader_1x15_P2.54mm_Vertical -> Connector_PinHeader_2.54mm:PinHeader_1x08_P2.54mm_Vertical
- moved J1 115.1 mm to (218.1, 84.6), turned to 180 degrees
- moved J2 88.9 mm to (192.7, 84.6), turned to 180 degrees
Connections:
- net /*D6 renamed DIO4
- net /A2 renamed DIO1
- net /A3 renamed DIO2
- net /A4/SDA renamed DIO3
- net /D7 renamed DIO5
- J1 pad 1: /D13/SCK -> GND
- J1 pad 2: +3V3 -> GND
- J1 pad 3: /AREF -> +3.3V
- J1 pad 4: /A0 -> LORA_RST
- J1 pad 5: /A1 -> DIO0
- J2 pad 1: /D12/MISO -> GND
- J2 pad 2: /*D11/MOSI -> CS
- J2 pad 3: /*D10/SS -> MOSI
- J2 pad 4: /*D9 -> MISO
- J2 pad 5: /D8 -> SCK
- J2 pad 8: /*D5 -> GND
Routing:
- net GND: track 0.00 -> 182.3 mm
- net SCL: track 0.00 -> 121.2 mm, vias 0 -> 2
- net SDA: track 0.00 -> 115.1 mm
- net +3.3V: track 0.00 -> 111.1 mm, vias 0 -> 1
- net TX: track 0.00 -> 95.2 mm, vias 0 -> 2
- net CS: track 0.00 -> 85.6 mm
- net RX: track 0.00 -> 78.1 mm, vias 0 -> 1
- net MISO: track 0.00 -> 68.0 mm
- net SCK: track 0.00 -> 66.4 mm
- net Net-(BT1--): track 0.00 -> 52.4 mm, vias 0 -> 1
- net MOSI: track 0.00 -> 48.1 mm, vias 0 -> 1
- net +BATT: track 0.00 -> 30.0 mm
- net LORA_RST: track 0.00 -> 28.1 mm
- net DIO0: track 0.00 -> 23.6 mm
- net LED: track 0.00 -> 22.5 mm
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- added copper zone on B.Cu, net GND
- added copper zone on F.Cu, net GND
Other:
- board size 43.2 x 17.8 mm -> 65.5 x 60.8 mm
- board text added: "+"
- board text added: "-"
- board text added: "ATGM336H"
- board text added: "Antenna hole"
- board text added: "Designed by Charlie Nicholson, July 2024"
- board text added: "Licensed under CERN-OHL-S-2.0"
- board text added: "LoRa"
- board text added: "MPU-9250"
- board text added: "Made possible by NESciTech, New England Weather Balloon Society, and Hack Club."
- board text added: "Mounting hole"
- board text added: "NEWbs"
- board text added: "OLED"
- board text added: "StratoSoar MK3 Ground Station LoRa telemetry receiver"
- board text added: "https://github.com/crnicholson/StratoSoar-MK3"
- board text removed: "ICSP"
- board text removed: "USB Mini-B"

Commit message: Commit
Other:
- board text added: "JLCJLCJLCJLC"
Changed lines of the file:
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@@
 		(layer "Edge.Cuts")
+	)
+	(gr_text "JLCJLCJLCJLC"
+		(at 225.552 123.571 -0)
+		(layer "B.SilkS")
+		(effects
+			(font
+				(size 1 1)
+				(thickness 0.15)
+			)
+			(justify left bottom mirror)
+		)
 	)
 	(gr_text "LoRa"
